File: M8HeadlessStaging/M8HeadlessStaging.sch (KiCad schematic (older format))
At the start: 10 parts, among them J1 MIDI OUT, J2 MIDI IN, U1 6N138, U1 Teensy4.1

Commit message: Add schematic
Parts:
- added J3: Key_frontpanel, symbol Connector:Conn_01x10_Male
- added J4: Key_raspiGPIO, symbol Connector:Conn_01x10_Female
- added SW1: UP, keyswitches:SW_PG1350, symbol Switch:SW_Push
- added SW2: DOWN, keyswitches:SW_PG1350, symbol Switch:SW_Push
- added SW3: RIGHT, keyswitches:SW_PG1350, symbol Switch:SW_Push
- added SW4: LEFT, keyswitches:SW_PG1350, symbol Switch:SW_Push
- added SW5: SHIFT, keyswitches:SW_PG1350, symbol Switch:SW_Push
- added SW6: PLAY, keyswitches:SW_PG1350, symbol Switch:SW_Push
- added SW7: OPTION, keyswitches:SW_PG1350, symbol Switch:SW_Push
- added SW8: EDIT, keyswitches:SW_PG1350, symbol Switch:SW_Push
- added U2: Raspberry_Pi_2_3, symbol Connector:Raspberry_Pi_2_3
Connections:
- net GND: now also J3.10 (Pin_10), J3.9 (Pin_9), J4.10 (Pin_10), J4.9 (Pin_9), SW1.1, SW2.1, SW3.1, SW4.1, SW5.1, SW6.1, SW7.1, SW8.1
- new net DOWN: J3.2 (Pin_2), J4.2 (Pin_2), SW2.2
- new net EDIT: J3.8 (Pin_8), J4.8 (Pin_8), SW8.2
- new net LEFT: J3.4 (Pin_4), J4.4 (Pin_4), SW4.2
- new net OPTION: J3.7 (Pin_7), J4.7 (Pin_7), SW7.2
- new net PLAY: J3.6 (Pin_6), J4.6 (Pin_6), SW6.2
- new net RIGHT: J3.3 (Pin_3), J4.3 (Pin_3), SW3.2
- new net SHIFT: J3.5 (Pin_5), J4.5 (Pin_5), SW5.2
- new net UP: J3.1 (Pin_1), J4.1 (Pin_1), SW1.2
Other:
- moved on the sheet: C1, D1, J1, J2, R1, R2, R3, R4, U1

Commit message: add schematics
Parts:
- removed J4: Key_raspiGPIO, symbol Connector:Conn_01x10_Female
- J3: footprint (none) -> Connector_PinHeader_2.54mm:PinHeader_2x05_P2.54mm_Vertical_SMD
Changed lines of the file:
@@
 	0    1    1    0
 $EndComp
-Text GLabel 7500 4150 2    50   Input ~ 0
-UP
 Text GLabel 8500 4150 2    50   Input ~ 0
 DOWN
@@
 Text GLabel 10550 4700 2    50   Input ~ 0
 EDIT
-$Comp
-L Connector:Conn_01x10_Female J4
-U 1 1 6188BFA7
-P 9100 5650
-F 0 "J4" H 9000 6300 50  0000 C CNN
-F 1 "Key_raspiGPIO" H 9000 6200 50  0000 C CNN
-F 2 "" H 9100 5650 50  0001 C CNN
-F 3 "~" H 9100 5650 50  0001 C CNN
-	1    9100 5650
-	-1   0    0    -1
-$EndComp
-$Comp
-L Connector:Conn_01x10_Male J3
-U 1 1 6188A148
-P 8500 5650
-F 0 "J3" H 8650 6300 50  0000 R CNN
-F 1 "Key_frontpanel" H 8850 6200 50  0000 R CNN
-F 2 "" H 8500 5650 50  0001 C CNN
-F 3 "~" H 8500 5650 50  0001 C CNN
-	1    8500 5650
-	-1   0    0    -1
-$EndComp
 Text GLabel 8300 5250 0    50   Input ~ 0
 UP
@@
 Text GLabel 8300 5950 0    50   Input ~ 0
 EDIT
-$Comp
-L power:GND #PWR?
-U 1 1 6189A4B2
-P 8300 6150
-F 0 "#PWR?" H 8300 5900 50  0001 C CNN
-F 1 "GND" V 8305 6022 50  0000 R CNN
-F 2 "" H 8300 6150 50  0001 C CNN
-F 3 "" H 8300 6150 50  0001 C CNN
-	1    8300 6150
-	0    1    1    0
-$EndComp
 Wire Wire Line
 	8300 6050 8300 6150
-Connection ~ 8300 6150
-Wire Wire Line
-	9300 6050 9300 6150
 $Comp
-L power:GND #PWR?
-U 1 1 6189C06B
-P 9300 6150
-F 0 "#PWR?" H 9300 5900 50  0001 C CNN
-F 1 "GND" V 9305 6022 50  0000 R CNN
-F 2 "" H 9300 6150 50  0001 C CNN
-F 3 "" H 9300 6150 50  0001 C CNN
-	1    9300 6150
-	0    -1   -1   0
+L Connector:Conn_01x10_Male J3
+U 1 1 6188A148
+P 8500 5650
+F 0 "J3" H 8650 6300 50  0000 R CNN
+F 1 "Key_frontpanel" H 8850 6200 50  0000 R CNN
+F 2 "Connector_PinHeader_2.54mm:PinHeader_2x05_P2.54mm_Vertical_SMD" H 8500 5650 50  0001 C CNN
+F 3 "~" H 8500 5650 50  0001 C CNN
+	1    8500 5650
+	-1   0    0    -1
 $EndComp
-Connection ~ 9300 6150
-Text GLabel 9300 5950 2    50   Input ~ 0
-EDIT
-Text GLabel 9300 5850 2    50   Input ~ 0
-OPTION
-Text GLabel 9300 5750 2    50   Input ~ 0
-PLAY
-Text GLabel 9300 5650 2    50   Input ~ 0
-SHIFT
-Text GLabel 9300 5550 2    50   Input ~ 0
-LEFT
-Text GLabel 9300 5450 2    50   Input ~ 0
-RIGHT
-Text GLabel 9300 5350 2    50   Input ~ 0
-DOWN
-Text GLabel 9300 5250 2    50   Input ~ 0
+Text GLabel 8300 6150 0    50   Input ~ 0
+GND
+Text GLabel 7500 4150 2    50   Input ~ 0
 UP
 $EndSCHEMATC
