File: M8HeadlessStaging/M8HeadlessStaging.sch (KiCad schematic (older format))
At the start: 20 parts, among them J1 MIDI OUT, J2 MIDI IN, J3 Key_frontpanel, SW1 UP, SW2 DOWN, SW3 RIGHT, SW4 LEFT, SW5 SHIFT, SW6 PLAY, SW7 OPTION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

Commit message: Add PCB
Parts:
- added J4: TO_RASP_VIN, MountingHole:MountingHole_3.2mm_M3, symbol Connector:Conn_01x01_Male
- added J5: TO_BAT_MODULE, MountingHole:MountingHole_3.2mm_M3, symbol Connector:Conn_01x01_Male
- added S1: SLIDE_SWITCH, digikey-footprints:Switch_Slide_11.6x4mm_EG1218, symbol dk_Slide-Switches:EG1218
- J1, J2: footprint (none) -> Connector_Audio:Jack_3.5mm_PJ311_Horizontal
- U1: footprint (none) -> digikey-footprints:TEENSY4.1
- U3: renamed from U1; footprint (none) -> Package_SO:SOP-8_6.62x9.15mm_P2.54mm
Connections:
- new net: J5.1 (Pin_1), S1.1
- new net: J4.1 (Pin_1), S1.2
- no-connect marks 1 -> 2
Changed lines of the file:
@@
 F 0 "U1" H 1850 5815 50  0000 C CNN
 F 1 "Teensy4.1" H 1850 5724 50  0000 C CNN
-F 2 "" H 1450 3650 50  0001 C CNN
+F 2 "digikey-footprints:TEENSY4.1" H 1450 3650 50  0001 C CNN
 F 3 "" H 1450 3650 50  0001 C CNN
 	1    1850 3250
@@
 F 0 "J1" H 4570 1883 50  0000 R CNN
 F 1 "MIDI OUT" H 4570 1974 50  0000 R CNN
-F 2 "" H 4850 1950 50  0001 C CNN
+F 2 "Connector_Audio:Jack_3.5mm_PJ311_Horizontal" H 4850 1950 50  0001 C CNN
 F 3 "~" H 4850 1950 50  0001 C CNN
 	1    4850 1950
@@
 $EndComp
 $Comp
-L power:GND #PWR?
+L power:GND #PWR0101
 U 1 1 61846E3E
 P 4650 2050
-F 0 "#PWR?" H 4650 1800 50  0001 C CNN
+F 0 "#PWR0101" H 4650 1800 50  0001 C CNN
 F 1 "GND" H 4655 1877 50  0000 C CNN
 F 2 "" H 4650 2050 50  0001 C CNN
@@
 F 0 "J2" H 3470 3033 50  0000 R CNN
 F 1 "MIDI IN" H 3470 3124 50  0000 R CNN
-F 2 "" H 3750 3100 50  0001 C CNN
+F 2 "Connector_Audio:Jack_3.5mm_PJ311_Horizontal" H 3750 3100 50  0001 C CNN
 F 3 "~" H 3750 3100 50  0001 C CNN
 	1    3750 3100
@@
 $EndComp
 $Comp
-L power:GND #PWR?
+L power:GND #PWR0102
 U 1 1 6184B62D
 P 3950 3000
-F 0 "#PWR?" H 3950 2750 50  0001 C CNN
+F 0 "#PWR0102" H 3950 2750 50  0001 C CNN
 F 1 "GND" H 3955 2827 50  0000 C CNN
 F 2 "" H 3950 3000 50  0001 C CNN
@@
 $EndComp
 $Comp
-L Isolator:6N138 U1
+L Isolator:6N138 U3
 U 1 1 6184F018
 P 5100 3050
-F 0 "U1" H 5100 3517 50  0000 C CNN
+F 0 "U3" H 5100 3517 50  0000 C CNN
 F 1 "6N138" H 5100 3426 50  0000 C CNN
-F 2 "" H 5390 2750 50  0001 C CNN
+F 2 "Package_SO:SOP-8_6.62x9.15mm_P2.54mm" H 5390 2750 50  0001 C CNN
 F 3 "http://www.onsemi.com/pub/Collateral/HCPL2731-D.pdf" H 5390 2750 50  0001 C CNN
 	1    5100 3050
@@
 	5700 2850 6100 2850
 $Comp
-L power:GND #PWR?
+L power:GND #PWR0103
 U 1 1 61852C15
 P 5700 2450
-F 0 "#PWR?" H 5700 2200 50  0001 C CNN
+F 0 "#PWR0103" H 5700 2200 50  0001 C CNN
 F 1 "GND" H 5705 2277 50  0000 C CNN
 F 2 "" H 5700 2450 50  0001 C CNN
@@
 	6000 3150 6100 3150
 $Comp
-L power:GND #PWR?
+L power:GND #PWR0104
 U 1 1 61855D65
 P 5600 3250
-F 0 "#PWR?" H 5600 3000 50  0001 C CNN
+F 0 "#PWR0104" H 5600 3000 50  0001 C CNN
 F 1 "GND" V 5605 3122 50  0000 R CNN
 F 2 "" H 5600 3250 50  0001 C CNN
@@
 $EndComp
 $Comp
-L power:GND #PWR?
+L power:GND #PWR0105
 U 1 1 6186D6BF
 P 7100 4150
-F 0 "#PWR?" H 7100 3900 50  0001 C CNN
+F 0 "#PWR0105" H 7100 3900 50  0001 C CNN
 F 1 "GND" V 7105 4022 50  0000 R CNN
 F 2 "" H 7100 4150 50  0001 C CNN
@@
 $EndComp
 $Comp
-L power:GND #PWR?
+L power:GND #PWR0106
 U 1 1 61870B9A
 P 8100 4150
-F 0 "#PWR?" H 8100 3900 50  0001 C CNN
+F 0 "#PWR0106" H 8100 3900 50  0001 C CNN
 F 1 "GND" V 8105 4022 50  0000 R CNN
 F 2 "" H 8100 4150 50  0001 C CNN
@@
 $EndComp
 $Comp
-L power:GND #PWR?
+L power:GND #PWR0107
 U 1 1 61872138
 P 9100 4150
-F 0 "#PWR?" H 9100 3900 50  0001 C CNN
+F 0 "#PWR0107" H 9100 3900 50  0001 C CNN
 F 1 "GND" V 9105 4022 50  0000 R CNN
 F 2 "" H 9100 4150 50  0001 C CNN
@@
 $EndComp
 $Comp
-L power:GND #PWR?
+L power:GND #PWR0108
 U 1 1 618734D4
 P 10150 4150
-F 0 "#PWR?" H 10150 3900 50  0001 C CNN
+F 0 "#PWR0108" H 10150 3900 50  0001 C CNN
 F 1 "GND" V 10155 4022 50  0000 R CNN
 F 2 "" H 10150 4150 50  0001 C CNN
@@
 $EndComp
 $Comp
-L power:GND #PWR?
+L power:GND #PWR0109
 U 1 1 618746B6
 P 7100 4700
-F 0 "#PWR?" H 7100 4450 50  0001 C CNN
+F 0 "#PWR0109" H 7100 4450 50  0001 C CNN
 F 1 "GND" V 7105 4572 50  0000 R CNN
 F 2 "" H 7100 4700 50  0001 C CNN
@@
 $EndComp
 $Comp
-L power:GND #PWR?
+L power:GND #PWR0110
 U 1 1 618746CA
 P 8100 4700
-F 0 "#PWR?" H 8100 4450 50  0001 C CNN
+F 0 "#PWR0110" H 8100 4450 50  0001 C CNN
 F 1 "GND" V 8105 4572 50  0000 R CNN
 F 2 "" H 8100 4700 50  0001 C CNN
@@
 $EndComp
 $Comp
-L power:GND #PWR?
+L power:GND #PWR0111
 U 1 1 618746DE
 P 9100 4700
-F 0 "#PWR?" H 9100 4450 50  0001 C CNN
+F 0 "#PWR0111" H 9100 4450 50  0001 C CNN
 F 1 "GND" V 9105 4572 50  0000 R CNN
 F 2 "" H 9100 4700 50  0001 C CNN
@@
 $EndComp
 $Comp
-L power:GND #PWR?
+L power:GND #PWR0112
 U 1 1 618746F2
 P 10150 4700
-F 0 "#PWR?" H 10150 4450 50  0001 C CNN
+F 0 "#PWR0112" H 10150 4450 50  0001 C CNN
 F 1 "GND" V 10155 4572 50  0000 R CNN
 F 2 "" H 10150 4700 50  0001 C CNN
@@
 Text GLabel 2950 1300 2    50   Input ~ 0
 +3V3
+$Comp
+L dk_Slide-Switches:EG1218 S1
+U 1 1 618EDC10
+P 10100 2450
+F 0 "S1" V 10054 2594 50  0000 L CNN
+F 1 "SLIDE_SWITCH" V 10145 2594 50  0000 L CNN
+F 2 "digikey-footprints:Switch_Slide_11.6x4mm_EG1218" H 10300 2650 50  0001 L CNN
+F 3 "http://spec_sheets.e-switch.com/specs/P040040.pdf" H 10300 2750 60  0001 L CNN
+F 4 "EG1903-ND" H 10300 2850 60  0001 L CNN "Digi-Key_PN"
+F 5 "EG1218" H 10300 2950 60  0001 L CNN "MPN"
+F 6 "Switches" H 10300 3050 60  0001 L CNN "Category"
+F 7 "Slide Switches" H 10300 3150 60  0001 L CNN "Family"
+F 8 "http://spec_sheets.e-switch.com/specs/P040040.pdf" H 10300 3250 60  0001 L CNN "DK_Datasheet_Link"
+F 9 "/product-detail/en/e-switch/EG1218/EG1903-ND/101726" H 10300 3350 60  0001 L CNN "DK_Detail_Page"
+F 10 "SWITCH SLIDE SPDT 200MA 30V" H 10300 3450 60  0001 L CNN "Description"
+F 11 "E-Switch" H 10300 3550 60  0001 L CNN "Manufacturer"
+F 12 "Active" H 10300 3650 60  0001 L CNN "Status"
+	1    10100 2450
+	0    1    1    0
+$EndComp
+Wire Wire Line
+	10100 1900 10100 2250
+NoConn ~ 10000 2650
+$Comp
+L Connector:Conn_01x01_Male J4
+U 1 1 618F504C
+P 10100 1700
+F 0 "J4" V 10162 1744 50  0000 L CNN
+F 1 "TO_RASP_VIN" V 10253 1744 50  0000 L CNN
+F 2 "MountingHole:MountingHole_3.2mm_M3" H 10100 1700 50  0001 C CNN
+F 3 "~" H 10100 1700 50  0001 C CNN
+	1    10100 1700
+	0    1    1    0
+$EndComp
+$Comp
+L Connector:Conn_01x01_Male J5
+U 1 1 618F7C2D
+P 10200 2850
+F 0 "J5" V 10354 2762 50  0000 R CNN
+F 1 "TO_BAT_MODULE" V 10263 2762 50  0000 R CNN
+F 2 "MountingHole:MountingHole_3.2mm_M3" H 10200 2850 50  0001 C CNN
+F 3 "~" H 10200 2850 50  0001 C CNN
+	1    10200 2850
+	0    -1   -1   0
+$EndComp
 $EndSCHEMATC
